File: hardware/v1/_autosave-ollyfc.kicad_pcb (KiCad board)
At the start: 4 copper layers, 50 x 95 mm, 98 parts, among them J1 Conn_01x06, J10 Conn_01x03, J11 Conn_01x03, J13 Conn_01x05, J2 Conn_01x02, J3 Conn_01x03, J4 USB_C_Receptacle_USB2.0, J5 Conn_02x05_Odd_Even, J6 Conn_01x03, J7 Conn_01x03, J8 Conn_Coaxial, J9 Conn_01x03, Q1 AO3401A, Q2 MMBT3904, Q3 MMBT3904, Q4 MMBT3904, SW1 ACT/PASS, SW2 SW_Push, SW3 SW_Push, SW4 MODE1, SW5 MODE1, U1 AMS1117-3.3, U10 SRV05-4, U2 PCA9685BS, U3 STM32F411RETx, U4 LIS3MDL, U5 BMI088, U6 W25Q128JVS, U7 BMP388, U8 NEO-M8N, U9 TPS2113APW, Y1 X322516MLB4SI

Commit message: some hardware designs
Parts:
- BZ1: moved to B.Cu
- moved R26 26.3 mm to (7.00, 23.2)
- moved BZ1 4.85 mm to (8.50, 34.2), turned to 0 degrees
- moved Q4 0.70 mm to (8.75, 19.8), turned to 90 degrees
Routing:
- net BUZZER: track 0.00 -> 11.8 mm
- net Net-(Q4-B): track 0.00 -> 2.57 mm
Changed lines of the file:
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@@
   )
   (footprint "Package_TO_SOT_SMD:SOT-23" (layer "F.Cu")
-    (at 8.6875 20.45)
+    (at 8.75 19.75 90)
     (descr "SOT, 3 Pin (https://www.jedec.org/system/files/docs/to-236h.pdf variant AB), generated with kicad-footprint-generator ipc_gullwing_generator.py")
     (tags "SOT TO_SOT_SMD")
@@
     (property "ki_keywords" "NPN Transistor")
     (attr smd)
-    (fp_text reference "Q4" (at 0 -2.4) (layer "F.SilkS")
+    (fp_text reference "Q4" (at 0 -2.4 90) (layer "F.SilkS")
         (effects (font (size 1 1) (thickness 0.15)))
     )
-    (fp_text value "MMBT3904" (at 0 2.4) (layer "F.Fab")
+    (fp_text value "MMBT3904" (at 0 2.4 90) (layer "F.Fab")
         (effects (font (size 1 1) (thickness 0.15)))
     )
-    (fp_text user "${REFERENCE}" (at 0 0) (layer "F.Fab")
+    (fp_text user "${REFERENCE}" (at 0 0 90) (layer "F.Fab")
         (effects (font (size 0.32 0.32) (thickness 0.05)))
     )
@@
     (fp_line (start 0.65 1.45) (end -0.65 1.45)
       (stroke (width 0.1) (type solid)) (layer "F.Fab"))
-    (pad "1" smd roundrect (at -0.9375 -0.95) (size 1.475 0.6) (layers "F.Cu" "F.Paste" "F.Mask") (roundrect_rratio 0.25)
+    (pad "1" smd roundrect (at -0.9375 -0.95 90) (size 1.475 0.6) (layers "F.Cu" "F.Paste" "F.Mask") (roundrect_rratio 0.25)
       (net 42 "Net-(Q4-B)") (pinfunction "B") (pintype "input"))
-    (pad "2" smd roundrect (at -0.9375 0.95) (size 1.475 0.6) (layers "F.Cu" "F.Paste" "F.Mask") (roundrect_rratio 0.25)
+    (pad "2" smd roundrect (at -0.9375 0.95 90) (size 1.475 0.6) (layers "F.Cu" "F.Paste" "F.Mask") (roundrect_rratio 0.25)
       (net 81 "GND") (pinfunction "E") (pintype "passive"))
-    (pad "3" smd roundrect (at 0.9375 0) (size 1.475 0.6) (layers "F.Cu" "F.Paste" "F.Mask") (roundrect_rratio 0.25)
+    (pad "3" smd roundrect (at 0.9375 0 90) (size 1.475 0.6) (layers "F.Cu" "F.Paste" "F.Mask") (roundrect_rratio 0.25)
       (net 43 "Net-(BZ1-+)") (pinfunction "C") (pintype "passive"))
     (model "${KICAD6_3DMODEL_DIR}/Package_TO_SOT_SMD.3dshapes/SOT-23.wrl"
@@
   )
   (footprint "Resistor_SMD:R_0603_1608Metric" (layer "F.Cu")
-    (at 31.9475 14.97)
+    (at 7 23.25)
     (descr "Resistor SMD 0603 (1608 Metric), square (rectangular) end terminal, IPC_7351 nominal, (Body size source: IPC-SM-782 page 72, https://www.pcb-3d.com/wordpress/wp-content/uploads/ipc-sm-782a_amendment_1_and_2.pdf), generated with kicad-footprint-generator")
     (tags "resistor")
@@
     )
   )
-  (footprint "Buzzer_Beeper:XDCR_CMT-9648-85T" (layer "F.Cu")
-    (at 3.75 35.25 135)
-    (property "Sheetfile" "sensor.kicad_sch")
-    (property "Sheetname" "IO")
-    (property "dnp" "")
-    (property "ki_description" "Buzzer, polarized")
-    (property "ki_keywords" "quartz resonator ceramic")
-    (attr through_hole)
-    (fp_text reference "BZ1" (at -0.325 -5.635 135) (layer "F.SilkS")
-        (effects (font (size 1 1) (thickness 0.15)))
-    )
-    (fp_text value "CMT-9648-85T" (at 7.195 5.465 135) (layer "F.Fab")
-        (effects (font (size 1 1) (thickness 0.15)))
-    )
-    (fp_text user "-" (at 5.2 0.4 135) (layer "F.SilkS")
-        (effects (font (size 1 1) (thickness 0.15)))
-    )
-    (fp_text user "+" (at -6 0.6 135) (layer "F.SilkS")
-        (effects (font (size 1 1) (thickness 0.15)))
-    )
-    (fp_text user "+" (at -6 0.6 135) (layer "F.Fab")
-        (effects (font (size 1 1) (thickness 0.15)))
-    )
-    (fp_text user "-" (at 5.2 0.4 135) (layer "F.Fab")
-        (effects (font (size 1 1) (thickness 0.15)))
-    )
-    (fp_circle (center 0 0) (end 4.5 0)
-      (stroke (width 0.127) (type solid)) (fill none) (layer "F.SilkS"))
-    (fp_circle (center 0 0) (end 4.75 0)
-      (stroke (width 0.05) (type solid)) (fill none) (layer "F.CrtYd"))
-    (fp_circle (center 0 0) (end 4.5 0)
-      (stroke (width 0.127) (type solid)) (fill none) (layer "F.Fab"))
-    (pad "N" thru_hole circle (at 2 0 135) (size 2 2) (drill 0.8) (layers "*.Cu" "*.Mask")
-      (solder_mask_margin 0.102))
-    (pad "P" thru_hole circle (at -2 0 135) (size 2 2) (drill 0.8) (layers "*.Cu" "*.Mask")
-      (solder_mask_margin 0.102))
-  )
   (footprint "Button_Switch_THT:SW_PUSH_6mm" (layer "F.Cu")
     (at -21.5 17.75 90)
@@
     )
   )
+  (footprint "Buzzer_Beeper:XDCR_CMT-9648-85T" (layer "B.Cu")
+    (at 8.5 34.25)
+    (property "Sheetfile" "sensor.kicad_sch")
+    (property "Sheetname" "IO")
+    (property "dnp" "")
+    (property "ki_description" "Buzzer, polarized")
+    (property "ki_keywords" "quartz resonator ceramic")
+    (attr through_hole)
+    (fp_text reference "BZ1" (at -0.325 5.635) (layer "B.SilkS")
+        (effects (font (size 1 1) (thickness 0.15)) (justify mirror))
+    )
+    (fp_text value "CMT-9648-85T" (at 7.195 -5.465) (layer "B.Fab")
+        (effects (font (size 1 1) (thickness 0.15)) (justify mirror))
+    )
+    (fp_text user "-" (at 5.2 -0.4) (layer "B.SilkS")
+        (effects (font (size 1 1) (thickness 0.15)) (justify mirror))
+    )
+    (fp_text user "+" (at -6 -0.6) (layer "B.SilkS")
+        (effects (font (size 1 1) (thickness 0.15)) (justify mirror))
+    )
+    (fp_text user "+" (at -6 -0.6) (layer "B.Fab")
+        (effects (font (size 1 1) (thickness 0.15)) (justify mirror))
+    )
+    (fp_text user "-" (at 5.2 -0.4) (layer "B.Fab")
+        (effects (font (size 1 1) (thickness 0.15)) (justify mirror))
+    )
+    (fp_circle (center 0 0) (end 4.5 0)
+      (stroke (width 0.127) (type solid)) (fill none) (layer "B.SilkS"))
+    (fp_circle (center 0 0) (end 4.75 0)
+      (stroke (width 0.05) (type solid)) (fill none) (layer "B.CrtYd"))
+    (fp_circle (center 0 0) (end 4.5 0)
+      (stroke (width 0.127) (type solid)) (fill none) (layer "B.Fab"))
+    (pad "N" thru_hole circle (at 2 0) (size 2 2) (drill 0.8) (layers "*.Cu" "*.Mask")
+      (solder_mask_margin 0.102))
+    (pad "P" thru_hole circle (at -2 0) (size 2 2) (drill 0.8) (layers "*.Cu" "*.Mask")
+      (solder_mask_margin 0.102))
+  )
   (footprint "Package_SO:SOIC-8_5.23x5.23mm_P1.27mm" (layer "B.Cu")
     (at -18 -5 180)
@@
   (segment (start 7.169239 -5.25) (end 7.75 -5.25) (width 0.2) (layer "B.Cu") (net 41))
   (segment (start 6.75 -5.25) (end 7.169239 -5.25) (width 0.2) (layer "B.Cu") (net 41))
+  (segment (start 7.825 23.25) (end 7.825 20.7125) (width 0.3) (layer "F.Cu") (net 42))
+  (segment (start 7.825 20.7125) (end 7.8 20.6875) (width 0.3) (layer "F.Cu") (net 42))
   (segment (start 6.75 -4.25) (end 5.275394 -2.775394) (width 0.2) (layer "F.Cu") (net 44))
   (segment (start 5.275394 -2.775394) (end 5.250268 -2.775394) (width 0.2) (layer "F.Cu") (net 44))
@@
   (segment (start -2.5 9.5) (end -4.7 11.7) (width 0.2) (layer "B.Cu") (net 55))
   (segment (start -3.75 19.35) (end -3 18.6) (width 0.2) (layer "B.Cu") (net 55))
+  (segment (start 6.5 20.25) (end 7 19.75) (width 0.2) (layer "F.Cu") (net 56))
+  (segment (start 7 19.75) (end 7 11.75) (width 0.2) (layer "F.Cu") (net 56))
+  (segment (start 6.175 23.25) (end 6.175 20.575) (width 0.2) (layer "F.Cu") (net 56))
+  (segment (start 6.175 20.575) (end 6.5 20.25) (width 0.2) (layer "F.Cu") (net 56))
   (segment (start 8.977984 -6.103484) (end 8.977984 -3.477984) (width 0.2) (layer "F.Cu") (net 59))
   (segment (start 0.5 -18) (end -1 -19.5) (width 0.2) (layer "F.Cu") (net 59))
